File: drone/PCB/dronePcb/dronePcb.kicad_sch (KiCad schematic)
At the start: 22 parts, among them M1 Motor_DC, M3 Motor_DC, M4 Motor_DC, Q1 PN2222A, Q2 PN2222A, Q3 PN2222A, Q4 PN2222A, SW1 SW_DPST_x2, U1 XIAO-ESP32-C6-DIP

Commit message: 改版
Parts:
- removed BT1: 3.3v, symbol Device:Battery_Cell
- removed D5: LED, symbol Device:LED
- removed R5: 220Ω, symbol Device:R
- BT2: value 5v -> 3.3v
Connections:
- net at D1.1 (K), D2.1 (K), D3.1 (K)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: now also SW1.1 (A), U1.12 (3V3)
- net at U1.14 (VBUS): no longer SW1.1 (A)
- no-connect marks 6 -> 8
