File: drone/PCB/dronePcb/dronePcb.kicad_sch (KiCad schematic)
At the start: 22 parts, among them M1 Motor_DC, M3 Motor_DC, M4 Motor_DC, Q1 PN2222A, Q2 PN2222A, Q3 PN2222A, Q4 PN2222A, SW1 SW_DPST_x2, U1 XIAO-ESP32-C6-DIP

Commit message: modify error
Parts:
- removed SW1: SW_DPST_x2, symbol Switch:SW_DPST_x2
- added SW1: SW_SPST, symbol Switch:SW_SPST
- M2: value ~ -> (none)
Connections:
- net at U1.14 (VBUS): now also SW1.1 (A)
- net at BT2.1 (+): now also SW1.2 (B)
- no-connect marks 6 -> 7
